File: electrical/CircuitPythonukiah.kicad_sch (KiCad schematic)
At the start: 22 parts, among them J1 USB_B_Micro, SW1 SW_DIP_x01, U1 QT_Py

Commit message: Update PCB schematic info
Other:
- title: (none) -> PCB, CircuitPythonukiah
Changed lines of the file:
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@@
 (kicad_sch (version 20211123) (generator eeschema)
   (paper "A4")
+  (title_block
+    (title "PCB, CircuitPythonukiah")
+    (date "2022-10-13")
+    (rev "1.0.0")
+    (comment 1 "Licensed under CERN-OHL-S version 2")
+    (comment 2 "Copyright Alec Delaney, 2022")
+  )
   (wire (pts (xy 127 151.13) (xy 130.81 151.13))
     (stroke (width 0) (type default) (color 0 0 0 0))
