File: electrical/CircuitPythonukiah.kicad_pcb (KiCad board)
At the start: 2 copper layers, 193 x 169 mm, 24 parts, among them J1 USB_B_Micro, M5 MountingHole_5.3mm_M5, SW1 SW_DIP_x01, U1 QT_Py

Commit message: Add OSHWA mark to PCB
Parts:
- added G***: LOGO, CircuitPythonukiah:OSHWA Mark, B.Cu at (128.3, 109.2)
